File: KiBoxLite_H/KiBoxLite_H.kicad_sch (KiCad schematic)
At the start: 151 parts, among them J1 Screw_Terminal_01x03, J2 USB_C_Receptacle_USB2.0_14P, Q2 BC817-40(SOT23), Q3 BC817-40(SOT23), T1 LMUN2211LT1G(SOT-23), U1 CH340X(MSOP-10), U10 MAX13487, U3 TP4054-42-SOT25-R(SOT23-5), U4 LAN8710A-EZC(QFN32), U5 TX4138(ESOIC-8)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

Commit message: build: USB-C Connected
Parts:
- removed J2: USB_C_Receptacle_USB2.0_14P, Connector_USB:USB_C_Receptacle_G-Switch_GT-USB-7025, symbol Connector:USB_C_Receptacle_USB2.0_14P
- added J2: USB4105-GF-A-060, Connector_USB:USB_C_Receptacle_GCT_USB4105-xx-A_16P_TopMnt_Horizontal, symbol USB4105-GF-A-060:USB4105-GF-A-060
Connections:
- net D+: now also J2.A6 (DP1), J2.B6 (DP2)
- net D-: now also J2.A7 (DN1), J2.B7 (DN2)
- net GND: now also L7.1, R63.1, J2.A1_B12 (GND), J2.B1_A12 (GND), J2.SH1 (SHELL_GND), J2.SH2 (SHELL_GND), J2.SH3 (SHELL_GND), J2.SH4 (SHELL_GND); no longer R63.2
- net GPI36\U1RXD: now also D10.1 (K), R23.1
- net at R62.1: now also J2.B5 (CC2)
- net +5V_USB renamed VBUS
- net VBUS: now also J2.A4_B9 (VBUS), J2.B4_A9 (VBUS)
- new net: J2.A5 (CC1), R63.2
- no-connect marks 15 -> 17
Other:
- moved on the sheet: C7, C8, L7, R62, R63
